File: Hak5-unify.kicad_pcb (KiCad board)
At the start: 2 copper layers, 27.3 x 17.5 mm, 4 parts, among them J1 Conn_01x02, J2 Conn_01x03, U1 Unify-Nano

Commit message: v0.4.1
Other:
- board size 27.3 x 17.5 mm -> 26 x 17.5 mm
- board text added: "v0.4.1"
- board text removed: "v0.4.0"
Changed lines of the file:
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@@
   (general
     (thickness 1.6)
-    (drawings 23)
+    (drawings 22)
     (tracks 18)
     (zones 0)
@@
     (0 F.Cu signal)
     (31 B.Cu signal)
-    (32 B.Adhes user hide)
-    (33 F.Adhes user hide)
-    (34 B.Paste user hide)
-    (35 F.Paste user hide)
+    (32 B.Adhes user)
+    (33 F.Adhes user)
+    (34 B.Paste user)
+    (35 F.Paste user)
     (36 B.SilkS user)
     (37 F.SilkS user)
-    (38 B.Mask user hide)
-    (39 F.Mask user hide)
-    (40 Dwgs.User user hide)
-    (41 Cmts.User user hide)
-    (42 Eco1.User user hide)
-    (43 Eco2.User user hide)
+    (38 B.Mask user)
+    (39 F.Mask user)
+    (40 Dwgs.User user)
+    (41 Cmts.User user)
+    (42 Eco1.User user)
+    (43 Eco2.User user)
     (44 Edge.Cuts user)
-    (45 Margin user hide)
-    (46 B.CrtYd user hide)
-    (47 F.CrtYd user hide)
-    (48 B.Fab user hide)
-    (49 F.Fab user hide)
+    (45 Margin user)
+    (46 B.CrtYd user)
+    (47 F.CrtYd user)
+    (48 B.Fab user)
+    (49 F.Fab user)
   )
   (setup
@@
     (pad_to_mask_clearance 0.2)
     (aux_axis_origin 0 0)
-    (visible_elements FFFFFF7F)
+    (visible_elements FFFFF77F)
     (pcbplotparams
       (layerselection 0x01030_ffffffff)
@@
       (effects (font (size 1 1) (thickness 0.15)))
     )
-    (fp_text value Unify-Nano (at 7 1) (layer F.Fab)
+    (fp_text value Unify-Nano (at 7.05 -0.95) (layer F.Fab)
       (effects (font (size 1 1) (thickness 0.15)))
     )
@@
     )
   )
-  (gr_line (start 121.7 82.5) (end 123 83.9) (layer Edge.Cuts) (width 0.2))
-  (gr_line (start 123 89.2) (end 123 83.9) (layer Edge.Cuts) (width 0.2))
-  (gr_line (start 127.34 89.2) (end 123 89.2) (layer Edge.Cuts) (width 0.2))
-  (gr_line (start 123 98) (end 121.1 100) (layer Edge.Cuts) (width 0.2))
+  (gr_line (start 122.85 95.9) (end 124.05 94.8) (layer Edge.Cuts) (width 0.2))
+  (gr_line (start 124.05 94.8) (end 125.95 94.8) (layer Edge.Cuts) (width 0.2))
+  (gr_line (start 124.6 82.5) (end 126 84) (layer Edge.Cuts) (width 0.2))
+  (gr_line (start 122.8 98.5) (end 121.35 100) (layer Edge.Cuts) (width 0.2))
   (gr_text "Designed by Spencer in Utah" (at 113.45 98.95) (layer B.SilkS)
     (effects (font (size 0.65 0.65) (thickness 0.1625)) (justify mirror))
@@
   (gr_line (start 100 84.5) (end 101.9 82.5) (layer Edge.Cuts) (width 0.2))
   (gr_line (start 100 97.6) (end 102.1 100) (layer Edge.Cuts) (width 0.2))
-  (gr_line (start 123 95.2) (end 123 97.9) (layer Edge.Cuts) (width 0.2))
-  (gr_line (start 127.34 95.1) (end 123 95.1) (layer Edge.Cuts) (width 0.2))
+  (gr_line (start 122.8 95.95) (end 122.8 98.45) (layer Edge.Cuts) (width 0.2))
   (gr_text "Cut Out" (at 112.8 90.9) (layer F.SilkS)
     (effects (font (size 1.5 1.5) (thickness 0.3)))
   )
-  (gr_line (start 127.34 89.2) (end 127.34 95.1) (layer Edge.Cuts) (width 0.2))
+  (gr_line (start 126 84) (end 126 94.8) (layer Edge.Cuts) (width 0.2))
   (gr_line (start 100 84.5) (end 100 97.6) (layer Edge.Cuts) (width 0.2))
-  (gr_line (start 102.1 100) (end 121.1 100) (layer Edge.Cuts) (width 0.2))
-  (gr_text TX1 (at 123.4 94 90) (layer F.SilkS)
+  (gr_line (start 102.1 100) (end 121.35 100) (layer Edge.Cuts) (width 0.2))
+  (gr_text TX1 (at 123 93.6 90) (layer F.SilkS)
     (effects (font (size 0.5 0.5) (thickness 0.125)))
   )
@@
     (effects (font (size 0.65 0.65) (thickness 0.1625)))
   )
-  (gr_text "v0.4.0\n" (at 102.7 85.9 45) (layer F.SilkS)
+  (gr_text "v0.4.1\n" (at 102.7 85.9 45) (layer F.SilkS)
     (effects (font (size 0.8 0.8) (thickness 0.125)))
   )
@@
     (effects (font (size 0.7 0.7) (thickness 0.125)))
   )
-  (gr_line (start 101.9 82.5) (end 121.7 82.5) (layer Edge.Cuts) (width 0.2))
+  (gr_line (start 101.9 82.5) (end 124.55 82.5) (layer Edge.Cuts) (width 0.2))
   (gr_line (start 106 98) (end 120.8 98) (layer Edge.Cuts) (width 0.2))
   (gr_line (start 106 84.6) (end 106 97.9) (layer Edge.Cuts) (width 0.2))
@@
   (segment (start 101.6 96.2) (end 102.95 96.2) (width 0.5) (layer F.Cu) (net 2))
   (segment (start 104.14 86.36) (end 105.94999 86.36) (width 0.5) (layer F.Cu) (net 5))
-  (segment (start 104 84.6) (end 104 86.5) (width 0.5) (layer F.Cu) (net 5))
-  (segment (start 105.4 83.2) (end 104 84.6) (width 0.5) (layer F.Cu) (net 5))
-  (segment (start 121.2 83.2) (end 105.4 83.2) (width 0.5) (layer F.Cu) (net 5))
-  (segment (start 121.8 90.8) (end 121.8 83.8) (width 0.5) (layer F.Cu) (net 5))
-  (segment (start 124.439999 93.439999) (end 121.8 90.8) (width 0.5) (layer F.Cu) (net 5))
-  (segment (start 125.579999 93.439999) (end 124.439999 93.439999) (width 0.5) (layer F.Cu) (net 5))
   (segment (start 125.74 93.6) (end 125.579999 93.439999) (width 0.5) (layer F.Cu) (net 5))
-  (segment (start 121.8 83.8) (end 121.2 83.2) (width 0.5) (layer F.Cu) (net 5))
+  (segment (start 121.8 91.01) (end 124.39 93.6) (width 0.5) (layer F.Cu) (net 5))
+  (segment (start 105.4 83.2) (end 121.2 83.2) (width 0.5) (layer F.Cu) (net 5))
+  (segment (start 121.8 83.8) (end 121.8 91.01) (width 0.5) (layer F.Cu) (net 5))
+  (segment (start 121.2 83.2) (end 121.8 83.8) (width 0.5) (layer F.Cu) (net 5))
+  (segment (start 124.39 93.6) (end 125.74 93.6) (width 0.5) (layer F.Cu) (net 5))
+  (segment (start 104 84.6) (end 105.4 83.2) (width 0.5) (layer F.Cu) (net 5))
+  (segment (start 104 86.5) (end 104 84.6) (width 0.5) (layer F.Cu) (net 5))
   (segment (start 103.1 91) (end 105.87499 88.22501) (width 0.65) (layer F.Cu) (net 8))
   (segment (start 101.6 91) (end 103.1 91) (width 0.65) (layer F.Cu) (net 8))

Commit message: v0.6.0
Parts:
- added JP1: SolderJumper_2_Open, Jumper:SolderJumper-2_P1.3mm_Open_RoundedPad1.0x1.5mm, F.Cu at (100.4, 102.1)
- added Q2: PMV65UNER, Package_TO_SOT_SMD:SOT-23, B.Cu at (100.5, 103.6)
- added R2: 10K, Resistor_THT:R_Axial_DIN0204_L3.6mm_D1.6mm_P7.62mm_Horizontal, F.Cu at (118.7, 91.7)
- added R3: 10K, Resistor_THT:R_Axial_DIN0204_L3.6mm_D1.6mm_P7.62mm_Horizontal, F.Cu at (120.3, 97.0)
- added SW1: SW_Push, Capacitor_SMD:CP_Elec_3x5.3, F.Cu at (113.0, 89.2)
- J1: value Conn_01x02 -> Conn_01x04; footprint Pin_Headers:Pin_Header_Straight_1x02_Pitch2.54mm -> Pin_Headers:Pin_Header_Straight_1x04_Pitch2.54mm
- R1: value R -> 10K; footprint Resistors_ThroughHole:R_Axial_DIN0204_L3.6mm_D1.6mm_P7.62mm_Horizontal -> Resistor_THT:R_Axial_DIN0204_L3.6mm_D1.6mm_P7.62mm_Horizontal
- moved J1 6.53 mm to (122.4, 99.2)
- moved J2 6.53 mm to (98.2, 101.8)
- moved U1 6.53 mm to (102.8, 103.3)
- moved R1 6.44 mm to (100.5, 91.9)
Connections:
- J1 pad 2: Net-(J1-Pad2) -> RX
- U1 pad 6: +5V -> Net-(JP1-Pad1)
Routing:
- net Net-(Q2-Pad1): track 0.00 -> 24.9 mm
- net RX: track 0.00 -> 8.31 mm
- net Net-(JP1-Pad1): track 0.00 -> 5.35 mm, vias 0 -> 1
- net GND: track 4.77 -> 8.45 mm
- net +5V: track 4.47 -> 5.33 mm
- net Net-(SW1-Pad1): track 0.00 -> 0.66 mm
- net Net-(SW1-Pad2): track 0.00 -> 0.62 mm
- net Net-(J2-Pad3): track 5.42 -> 4.87 mm
- net TX: track 34.8 -> 35.3 mm
- net (no net): vias 0 -> 4
Other:
- board size 26 x 17.5 mm -> 27.1 x 17.5 mm
- board text added: "TX3"
- board text added: "v0.6.0"
- board text removed: "TX1"
- board text removed: "v0.4.1"

Commit message: 0.7.0
Parts:
- JP1: moved to B.Cu
- moved Q2 13.5 mm to (99.7, 90.2), turned to 180 degrees
- moved JP1 9.28 mm to (98.2, 93.1), turned to 0 degrees
- moved R3 6.00 mm to (120.2, 91.0), turned to 270 degrees
- moved R2 5.25 mm to (118.6, 96.9), turned to 90 degrees
- moved R1 1.18 mm to (100.5, 93.1)
Connections:
- JP1 pad 2: +5V -> GND
- Q2 pad 2: Net-(JP1-Pad1) -> GND
- Q2 pad 3: +5V -> Net-(JP1-Pad1)
- U1 pad 5: GND -> Net-(JP1-Pad1)
- U1 pad 6: Net-(JP1-Pad1) -> +5V
Routing:
- net GND: track 8.45 -> 42.4 mm
- net Net-(JP1-Pad1): track 5.35 -> 12.4 mm
- net RX: track 8.31 -> 2.97 mm
- net TX: track 35.3 -> 40.0 mm
- net Net-(Q2-Pad1): track 24.9 -> 20.7 mm
- net (no net): vias 4 -> 0
Other:
- board text added: "GND"
- board text added: "RX3"
- board text added: "Video"
- board text added: "v0.7.0"
- board text removed: "v0.6.0"
