File: Hak5-unify.sch (KiCad schematic (older format))
At the start: 5 parts, among them J1 Conn_01x04, J2 Conn_01x03, SW1 SW_Push, U1 Unify-Nano

Commit message: v0.1.1
Changed lines of the file:
@@
 L power:+5V #PWR04
 U 1 1 5B761343
-P 3150 2850
-F 0 "#PWR04" H 3150 2700 50  0001 C CNN
-F 1 "+5V" H 3150 2990 50  0000 C CNN
-F 2 "" H 3150 2850 50  0001 C CNN
-F 3 "" H 3150 2850 50  0001 C CNN
-	1    3150 2850
+P 3200 2900
+F 0 "#PWR04" H 3200 2750 50  0001 C CNN
+F 1 "+5V" H 3200 3040 50  0000 C CNN
+F 2 "" H 3200 2900 50  0001 C CNN
+F 3 "" H 3200 2900 50  0001 C CNN
+	1    3200 2900
 	0    -1   -1   0
-$EndComp
-$Comp
-L power:+5V #PWR05
-U 1 1 5B76136C
-P 3350 2450
-F 0 "#PWR05" H 3350 2300 50  0001 C CNN
-F 1 "+5V" H 3350 2590 50  0000 C CNN
-F 2 "" H 3350 2450 50  0001 C CNN
-F 3 "" H 3350 2450 50  0001 C CNN
-	1    3350 2450
-	-1   0    0    1
 $EndComp
 Text GLabel 6600 2650 0    60   Input ~ 0
@@
 Wire Wire Line
 	2900 3100 3200 3100
+$Comp
+L power:GND #PWR?
+U 1 1 5B7B8B77
+P 3350 2450
+F 0 "#PWR?" H 3350 2200 50  0001 C CNN
+F 1 "GND" H 3355 2277 50  0000 C CNN
+F 2 "" H 3350 2450 50  0001 C CNN
+F 3 "" H 3350 2450 50  0001 C CNN
+	1    3350 2450
+	1    0    0    -1
+$EndComp
 $EndSCHEMATC

Commit message: v0.3.0
Parts:
- added J3: Conn_01x01_Female, Connector_PinHeader_2.54mm:PinHeader_1x01_P2.54mm_Vertical, symbol Connector:Conn_01x01_Female
- R1: footprint Resistors_THT:R_Axial_DIN0204_L3.6mm_D1.6mm_P5.08mm_Horizontal -> (none)
Changed lines of the file:
@@
 F 0 "R1" V 3430 2300 50  0000 C CNN
 F 1 "R" V 3350 2300 50  0000 C CNN
-F 2 "Resistors_THT:R_Axial_DIN0204_L3.6mm_D1.6mm_P5.08mm_Horizontal" V 3280 2300 50  0001 C CNN
+F 2 "" V 3280 2300 50  0001 C CNN
 F 3 "" H 3350 2300 50  0001 C CNN
 	1    3350 2300
@@
 	2900 3100 3200 3100
 $Comp
-L power:GND #PWR?
+L power:GND #PWR0101
 U 1 1 5B7B8B77
 P 3350 2450
-F 0 "#PWR?" H 3350 2200 50  0001 C CNN
+F 0 "#PWR0101" H 3350 2200 50  0001 C CNN
 F 1 "GND" H 3355 2277 50  0000 C CNN
 F 2 "" H 3350 2450 50  0001 C CNN
@@
 	1    0    0    -1
 $EndComp
+$Comp
+L Connector:Conn_01x01_Female J3
+U 1 1 5B8F658D
+P 6350 1900
+F 0 "J3" H 6377 1926 50  0000 L CNN
+F 1 "Conn_01x01_Female" H 6377 1835 50  0000 L CNN
+F 2 "Connector_PinHeader_2.54mm:PinHeader_1x01_P2.54mm_Vertical" H 6350 1900 50  0001 C CNN
+F 3 "~" H 6350 1900 50  0001 C CNN
+	1    6350 1900
+	1    0    0    -1
+$EndComp

Commit message: 2holes
Parts:
- removed J3: Conn_01x01_Female, Connector_PinHeader_2.54mm:PinHeader_1x01_P2.54mm_Vertical, symbol Connector:Conn_01x01_Female
- removed SW1: SW_Push, symbol Switch:SW_Push
- J1: value Conn_01x04 -> Conn_01x02; footprint Pin_Headers:Pin_Header_Straight_1x04_Pitch2.54mm -> Pin_Headers:Pin_Header_Straight_1x02_Pitch2.54mm; symbol Hak5-unify-rescue:Conn_01x04 -> Connector:Conn_01x02_Male
- R1: footprint (none) -> Resistor_THT:R_Axial_DIN0207_L6.3mm_D2.5mm_P2.54mm_Vertical
Connections:
- net labels removed: RX
- wire segments 12 -> 8
Changed lines of the file:
@@
 F 0 "R1" V 3430 2300 50  0000 C CNN
 F 1 "R" V 3350 2300 50  0000 C CNN
-F 2 "" V 3280 2300 50  0001 C CNN
+F 2 "Resistor_THT:R_Axial_DIN0207_L6.3mm_D2.5mm_P2.54mm_Vertical" V 3280 2300 50  0001 C CNN
 F 3 "" H 3350 2300 50  0001 C CNN
 	1    3350 2300
@@
 $EndComp
 $Comp
-L Hak5-unify-rescue:Conn_01x04 J1
+L Connector:Conn_01x02_Male J1
 U 1 1 5B72F16A
-P 6800 2650
-F 0 "J1" H 6800 2850 50  0000 C CNN
-F 1 "Conn_01x04" H 6800 2350 50  0000 C CNN
-F 2 "Pin_Headers:Pin_Header_Straight_1x04_Pitch2.54mm" H 6800 2650 50  0001 C CNN
-F 3 "" H 6800 2650 50  0001 C CNN
-	1    6800 2650
-	1    0    0    -1
+P 6200 2650
+F 0 "J1" H 6200 2850 50  0000 C CNN
+F 1 "Conn_01x02" H 6200 2350 50  0000 C CNN
+F 2 "Pin_Headers:Pin_Header_Straight_1x02_Pitch2.54mm" H 6200 2650 50  0001 C CNN
+F 3 "" H 6200 2650 50  0001 C CNN
+	1    6200 2650
+	-1   0    0    1
 $EndComp
 $Comp
@@
 	1    0    0    -1
 $EndComp
-Text GLabel 6600 2550 0    60   Input ~ 0
+Text GLabel 6000 2650 0    60   Input ~ 0
 TX
 Text GLabel 3900 2550 0    60   Input ~ 0
@@
 	0    -1   -1   0
 $EndComp
-Text GLabel 6600 2650 0    60   Input ~ 0
-RX
 Wire Wire Line
 	3900 2150 3350 2150
-$Comp
-L Switch:SW_Push SW1
-U 1 1 5B778E01
-P 4900 1750
-F 0 "SW1" H 4900 2035 50  0000 C CNN
-F 1 "SW_Push" H 4900 1944 50  0000 C CNN
-F 2 "" H 4900 1950 50  0001 C CNN
-F 3 "" H 4900 1950 50  0001 C CNN
-	1    4900 1750
-	1    0    0    -1
-$EndComp
 $Comp
 L Hak5-unify-rescue:Unify-Nano U1
@@
 	1    0    0    -1
 $EndComp
-Wire Wire Line
-	5100 1750 5100 2300
-Wire Wire Line
-	5100 2300 4950 2300
-Wire Wire Line
-	4700 1750 4700 2300
-Wire Wire Line
-	4700 2300 4800 2300
 Wire Wire Line
 	4000 2650 3700 2650
@@
 	1    0    0    -1
 $EndComp
-$Comp
-L Connector:Conn_01x01_Female J3
-U 1 1 5B8F658D
-P 6350 1900
-F 0 "J3" H 6377 1926 50  0000 L CNN
-F 1 "Conn_01x01_Female" H 6377 1835 50  0000 L CNN
-F 2 "Connector_PinHeader_2.54mm:PinHeader_1x01_P2.54mm_Vertical" H 6350 1900 50  0001 C CNN
-F 3 "~" H 6350 1900 50  0001 C CNN
-	1    6350 1900
-	1    0    0    -1
-$EndComp

Commit message: v0.6.0
Parts:
- added JP1: SolderJumper_2_Open, Jumper:SolderJumper-2_P1.3mm_Open_RoundedPad1.0x1.5mm, symbol Jumper:SolderJumper_2_Open
- added Q2: PMV65UNER, Package_TO_SOT_SMD:SOT-23, symbol Transistor_FET:BSS138
- added R2, R3: 10K, Resistor_THT:R_Axial_DIN0204_L3.6mm_D1.6mm_P7.62mm_Horizontal, symbol Device:R
- added SW1: SW_Push, Capacitor_SMD:CP_Elec_3x5.3, symbol Switch:SW_Push
- J1: value Conn_01x02 -> Conn_01x04; footprint Pin_Headers:Pin_Header_Straight_1x02_Pitch2.54mm -> Pin_Headers:Pin_Header_Straight_1x04_Pitch2.54mm; symbol Connector:Conn_01x02_Male -> Connector:Conn_01x04_Male
- R1: value R -> 10K; footprint Resistor_THT:R_Axial_DIN0207_L6.3mm_D2.5mm_P2.54mm_Vertical -> Resistor_THT:R_Axial_DIN0204_L3.6mm_D1.6mm_P7.62mm_Horizontal
Connections:
- net labels added: RX
- wire segments 8 -> 17
Changed lines of the file:
@@
-$EndComp
-$Comp
-L power:+5V #PWR02
-U 1 1 5B726591
-P 4000 3050
-F 0 "#PWR02" H 4000 2900 50  0001 C CNN
-F 1 "+5V" H 4000 3190 50  0000 C CNN
-F 2 "" H 4000 3050 50  0001 C CNN
-F 3 "" H 4000 3050 50  0001 C CNN
-	1    4000 3050
-	0    -1   -1   0
 $EndComp
 $Comp
@@
 P 3350 2300
 F 0 "R1" V 3430 2300 50  0000 C CNN
-F 1 "R" V 3350 2300 50  0000 C CNN
-F 2 "Resistor_THT:R_Axial_DIN0207_L6.3mm_D2.5mm_P2.54mm_Vertical" V 3280 2300 50  0001 C CNN
+F 1 "10K" V 3350 2300 50  0000 C CNN
+F 2 "Resistor_THT:R_Axial_DIN0204_L3.6mm_D1.6mm_P7.62mm_Horizontal" V 3280 2300 50  0001 C CNN
 F 3 "" H 3350 2300 50  0001 C CNN
 	1    3350 2300
@@
 $EndComp
 $Comp
-L Connector:Conn_01x02_Male J1
+L Connector:Conn_01x04_Male J1
 U 1 1 5B72F16A
 P 6200 2650
 F 0 "J1" H 6200 2850 50  0000 C CNN
-F 1 "Conn_01x02" H 6200 2350 50  0000 C CNN
-F 2 "Pin_Headers:Pin_Header_Straight_1x02_Pitch2.54mm" H 6200 2650 50  0001 C CNN
+F 1 "Conn_01x04" H 6200 2350 50  0000 C CNN
+F 2 "Pin_Headers:Pin_Header_Straight_1x04_Pitch2.54mm" H 6200 2650 50  0001 C CNN
 F 3 "" H 6200 2650 50  0001 C CNN
 	1    6200 2650
@@
 	1    0    0    -1
 $EndComp
-Text GLabel 6000 2650 0    60   Input ~ 0
+Text GLabel 6000 2750 0    60   Input ~ 0
 TX
 Text GLabel 3900 2550 0    60   Input ~ 0
@@
 	0    1    1    0
 $EndComp
-$Comp
-L power:+5V #PWR04
-U 1 1 5B761343
-P 3200 2900
-F 0 "#PWR04" H 3200 2750 50  0001 C CNN
-F 1 "+5V" H 3200 3040 50  0000 C CNN
-F 2 "" H 3200 2900 50  0001 C CNN
-F 3 "" H 3200 2900 50  0001 C CNN
-	1    3200 2900
-	0    -1   -1   0
-$EndComp
 Wire Wire Line
 	3900 2150 3350 2150
@@
 	1    0    0    -1
 $EndComp
+Text GLabel 6000 2650 0    50   Input ~ 0
+RX
+Wire Wire Line
+	3900 3050 4000 3050
+$Comp
+L Device:R R2
+U 1 1 5B94BC43
+P 2850 4100
+F 0 "R2" V 2750 4100 50  0000 C CNN
+F 1 "10K" V 2850 4100 50  0000 C CNN
+F 2 "Resistor_THT:R_Axial_DIN0204_L3.6mm_D1.6mm_P7.62mm_Horizontal" V 2780 4100 50  0001 C CNN
+F 3 "~" H 2850 4100 50  0001 C CNN
+	1    2850 4100
+	-1   0    0    1
+$EndComp
+Text GLabel 2550 3950 0    50   Input ~ 0
+RX
+$Comp
+L Transistor_FET:BSS138 Q2
+U 1 1 5B986C0D
+P 3050 3950
+F 0 "Q2" H 3255 3996 50  0000 L CNN
+F 1 "PMV65UNER" H 3255 3905 50  0000 L CNN
+F 2 "Package_TO_SOT_SMD:SOT-23" H 3250 3875 50  0001 L CIN
+F 3 "https://www.fairchildsemi.com/datasheets/BS/BSS138.pdf" H 3050 3950 50  0001 L CNN
+	1    3050 3950
+	1    0    0    -1
+$EndComp
+$Comp
+L Device:R R3
+U 1 1 5B986D27
+P 2700 3950
+F 0 "R3" V 2600 3950 50  0000 C CNN
+F 1 "10K" V 2700 3950 50  0000 C CNN
+F 2 "Resistor_THT:R_Axial_DIN0204_L3.6mm_D1.6mm_P7.62mm_Horizontal" V 2630 3950 50  0001 C CNN
+F 3 "~" H 2700 3950 50  0001 C CNN
+	1    2700 3950
+	0    1    1    0
+$EndComp
+Wire Wire Line
+	2900 3700 3150 3700
+Wire Wire Line
+	3150 3700 3150 3750
+$Comp
+L power:GND #PWR0102
+U 1 1 5B987485
+P 2850 4250
+F 0 "#PWR0102" H 2850 4000 50  0001 C CNN
+F 1 "GND" H 2855 4077 50  0000 C CNN
+F 2 "" H 2850 4250 50  0001 C CNN
+F 3 "" H 2850 4250 50  0001 C CNN
+	1    2850 4250
+	1    0    0    -1
+$EndComp
+$Comp
+L power:+5V #PWR0103
+U 1 1 5B987653
+P 3200 2900
+F 0 "#PWR0103" H 3200 2750 50  0001 C CNN
+F 1 "+5V" V 3215 3028 50  0000 L CNN
+F 2 "" H 3200 2900 50  0001 C CNN
+F 3 "" H 3200 2900 50  0001 C CNN
+	1    3200 2900
+	0    -1   -1   0
+$EndComp
+$Comp
+L power:+5V #PWR0104
+U 1 1 5B9876B2
+P 2900 3700
+F 0 "#PWR0104" H 2900 3550 50  0001 C CNN
+F 1 "+5V" V 2915 3828 50  0000 L CNN
+F 2 "" H 2900 3700 50  0001 C CNN
+F 3 "" H 2900 3700 50  0001 C CNN
+	1    2900 3700
+	0    -1   -1   0
+$EndComp
+Connection ~ 2850 3950
+Wire Wire Line
+	3150 4150 3900 4150
+Wire Wire Line
+	3900 4150 3900 3050
+$Comp
+L power:+5V #PWR0105
+U 1 1 5B988E48
+P 6000 2550
+F 0 "#PWR0105" H 6000 2400 50  0001 C CNN
+F 1 "+5V" V 6015 2678 50  0000 L CNN
+F 2 "" H 6000 2550 50  0001 C CNN
+F 3 "" H 6000 2550 50  0001 C CNN
+	1    6000 2550
+	0    -1   -1   0
+$EndComp
+$Comp
+L power:GND #PWR0106
+U 1 1 5B988EAE
+P 6000 2450
+F 0 "#PWR0106" H 6000 2200 50  0001 C CNN
+F 1 "GND" V 6005 2322 50  0000 R CNN
+F 2 "" H 6000 2450 50  0001 C CNN
+F 3 "" H 6000 2450 50  0001 C CNN
+	1    6000 2450
+	0    1    1    0
+$EndComp
+$Comp
+L Jumper:SolderJumper_2_Open JP1
+U 1 1 5B98A042
+P 4050 4150
+F 0 "JP1" H 4050 4355 50  0000 C CNN
+F 1 "SolderJumper_2_Open" H 4400 4250 50  0000 C CNN
+F 2 "Jumper:SolderJumper-2_P1.3mm_Open_RoundedPad1.0x1.5mm" H 4050 4150 50  0001 C CNN
+F 3 "~" H 4050 4150 50  0001 C CNN
+	1    4050 4150
+	1    0    0    -1
+$EndComp
+Connection ~ 3900 4150
+$Comp
+L power:+5V #PWR0107
+U 1 1 5B98A0F2
+P 4200 4150
+F 0 "#PWR0107" H 4200 4000 50  0001 C CNN
+F 1 "+5V" V 4215 4278 50  0000 L CNN
+F 2 "" H 4200 4150 50  0001 C CNN
+F 3 "" H 4200 4150 50  0001 C CNN
+	1    4200 4150
+	0    1    1    0
+$EndComp
+$Comp
+L Switch:SW_Push SW1
+U 1 1 5B9EB406
+P 4850 2150
+F 0 "SW1" H 4850 2435 50  0000 C CNN
+F 1 "SW_Push" H 4850 2344 50  0000 C CNN
+F 2 "Capacitor_SMD:CP_Elec_3x5.3" H 4850 2350 50  0001 C CNN
+F 3 "" H 4850 2350 50  0001 C CNN
+	1    4850 2150
+	1    0    0    -1
+$EndComp
+Wire Wire Line
+	4950 2300 5050 2300
+Wire Wire Line
+	5050 2300 5050 2150
+Wire Wire Line
+	4800 2300 4650 2300
+Wire Wire Line
+	4650 2300 4650 2150
 $EndSCHEMATC

Commit message: 0.7.0
Parts:
- J2: symbol Hak5-unify-rescue:Conn_01x03 -> Hak5-unify-rescue:Conn_01x03-Hak5-unify-rescue
- U1: symbol Hak5-unify-rescue:Unify-Nano -> Hak5-unify-rescue:Unify-Nano-Hak5-unify-rescue
Connections:
- wire segments 17 -> 18
Changed lines of the file:
@@
 $EndDescr
-$Comp
-L power:GND #PWR01
-U 1 1 5B72656F
-P 4000 2950
-F 0 "#PWR01" H 4000 2700 50  0001 C CNN
-F 1 "GND" H 4000 2800 50  0000 C CNN
-F 2 "" H 4000 2950 50  0001 C CNN
-F 3 "" H 4000 2950 50  0001 C CNN
-	1    4000 2950
-	0    1    1    0
-$EndComp
 $Comp
 L Device:R R1
@@
 $EndComp
 $Comp
-L Hak5-unify-rescue:Conn_01x03 J2
+L Hak5-unify-rescue:Conn_01x03-Hak5-unify-rescue J2
 U 1 1 5B7500FF
 P 3400 3000
@@
 	3900 2150 3350 2150
 $Comp
-L Hak5-unify-rescue:Unify-Nano U1
+L Hak5-unify-rescue:Unify-Nano-Hak5-unify-rescue U1
 U 1 1 5B726417
 P 4700 3250
@@
 Text GLabel 6000 2650 0    50   Input ~ 0
 RX
-Wire Wire Line
-	3900 3050 4000 3050
 $Comp
 L Device:R R2
@@
 $EndComp
 Wire Wire Line
-	2900 3700 3150 3700
-Wire Wire Line
 	3150 3700 3150 3750
 $Comp
@@
 	0    -1   -1   0
 $EndComp
-$Comp
-L power:+5V #PWR0104
-U 1 1 5B9876B2
-P 2900 3700
-F 0 "#PWR0104" H 2900 3550 50  0001 C CNN
-F 1 "+5V" V 2915 3828 50  0000 L CNN
-F 2 "" H 2900 3700 50  0001 C CNN
-F 3 "" H 2900 3700 50  0001 C CNN
-	1    2900 3700
-	0    -1   -1   0
-$EndComp
 Connection ~ 2850 3950
-Wire Wire Line
-	3150 4150 3900 4150
-Wire Wire Line
-	3900 4150 3900 3050
 $Comp
 L power:+5V #PWR0105
@@
 	1    0    0    -1
 $EndComp
-Connection ~ 3900 4150
-$Comp
-L power:+5V #PWR0107
-U 1 1 5B98A0F2
-P 4200 4150
-F 0 "#PWR0107" H 4200 4000 50  0001 C CNN
-F 1 "+5V" V 4215 4278 50  0000 L CNN
-F 2 "" H 4200 4150 50  0001 C CNN
-F 3 "" H 4200 4150 50  0001 C CNN
-	1    4200 4150
-	0    1    1    0
-$EndComp
 $Comp
 L Switch:SW_Push SW1
@@
 Wire Wire Line
 	4650 2300 4650 2150
+Wire Wire Line
+	3900 2950 4000 2950
+Wire Wire Line
+	3900 2950 3900 3700
+$Comp
+L power:GND #PWR?
+U 1 1 5BC424FD
+P 4200 4150
+F 0 "#PWR?" H 4200 3900 50  0001 C CNN
+F 1 "GND" V 4205 4022 50  0000 R CNN
+F 2 "" H 4200 4150 50  0001 C CNN
+F 3 "" H 4200 4150 50  0001 C CNN
+	1    4200 4150
+	0    -1   -1   0
+$EndComp
+$Comp
+L power:GND #PWR?
+U 1 1 5BC4255C
+P 3150 4300
+F 0 "#PWR?" H 3150 4050 50  0001 C CNN
+F 1 "GND" V 3155 4172 50  0000 R CNN
+F 2 "" H 3150 4300 50  0001 C CNN
+F 3 "" H 3150 4300 50  0001 C CNN
+	1    3150 4300
+	1    0    0    -1
+$EndComp
+$Comp
+L power:+5V #PWR?
+U 1 1 5BC425D3
+P 4000 3050
+F 0 "#PWR?" H 4000 2900 50  0001 C CNN
+F 1 "+5V" H 4015 3223 50  0000 C CNN
+F 2 "" H 4000 3050 50  0001 C CNN
+F 3 "" H 4000 3050 50  0001 C CNN
+	1    4000 3050
+	-1   0    0    1
+$EndComp
+Wire Wire Line
+	3150 3700 3900 3700
+Connection ~ 3900 3700
+Wire Wire Line
+	3900 3700 3900 4150
+Wire Wire Line
+	3150 4150 3150 4300
 $EndSCHEMATC
